File: Rev A/DAC.kicad_sch (KiCad schematic)
At the start: 19 parts, among them U6 74HC595

Commit message: added more schematic stuffs
Changed lines of the file:
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@@
 			(effects
 				(font
-					(size 1.27 1.27)
+					(size 0.8 0.8)
 				)
 				(hide yes)
@@
 			(effects
 				(font
-					(size 1.27 1.27)
+					(size 0.8 0.8)
 				)
 			)
@@
 			(effects
 				(font
-					(size 1.27 1.27)
+					(size 0.8 0.8)
 				)
 				(hide yes)
@@
 			(effects
 				(font
-					(size 1.27 1.27)
+					(size 0.8 0.8)
 				)
 			)
@@
 			(effects
 				(font
-					(size 1.27 1.27)
+					(size 0.8 0.8)
 				)
 				(justify left)
@@
 			(effects
 				(font
-					(size 1.27 1.27)
+					(size 0.8 0.8)
 				)
 				(justify left)
@@
 			(effects
 				(font
-					(size 1.27 1.27)
+					(size 0.8 0.8)
 				)
 				(hide yes)
@@
 			(effects
 				(font
-					(size 1.27 1.27)
+					(size 0.8 0.8)
 				)
 			)
@@
 			(effects
 				(font
-					(size 1.27 1.27)
+					(size 0.8 0.8)
 				)
 				(justify left)
@@
 			(effects
 				(font
-					(size 1.27 1.27)
+					(size 0.8 0.8)
 				)
 				(justify left)
@@
 			(effects
 				(font
-					(size 1.27 1.27)
+					(size 0.8 0.8)
 				)
 				(hide yes)
@@
 			(effects
 				(font
-					(size 1.27 1.27)
+					(size 0.8 0.8)
 				)
 			)
@@
 			(effects
 				(font
-					(size 1.27 1.27)
+					(size 0.8 0.8)
 				)
 				(hide yes)
@@
 			(effects
 				(font
-					(size 1.27 1.27)
+					(size 0.8 0.8)
 				)
 			)
@@
 			(effects
 				(font
-					(size 1.27 1.27)
+					(size 0.8 0.8)
 				)
 				(justify left)
@@
 			(effects
 				(font
-					(size 1.27 1.27)
+					(size 0.8 0.8)
 				)
 				(justify left)

Commit message: routed
Parts:
- removed R19: 0805,0, R_0805_2012Metric, symbol jlcpcb-basic-resistor:0805,0
- U6: footprint (none) -> Package_DIP:DIP-16_W7.62mm_Socket
Connections:
- net GND: now also U6.13 (~{OE})
Changed lines of the file:
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@@
 	(wire
 		(pts
-			(xy 107.95 116.84) (xy 107.95 120.65)
+			(xy 107.95 116.84) (xy 107.95 130.81)
 		)
 		(stroke
@@
 		(pts
 			(xy 162.56 86.36) (xy 161.29 86.36)
-		)
-		(stroke
-			(width 0)
-			(type default)
-		)
-	)
-	(wire
-		(pts
-			(xy 107.95 125.73) (xy 107.95 130.81)
 		)
 		(stroke
@@
 	)
 	(symbol
-		(lib_id "jlcpcb-basic-resistor:0805,0")
-		(at 107.95 123.19 0)
-		(unit 1)
-		(exclude_from_sim no)
-		(in_bom yes)
-		(on_board yes)
-		(dnp no)
-		(fields_autoplaced yes)
-		(property "Reference" "R19"
-			(at 110.49 121.9199 0)
-			(effects
-				(font
-					(size 0.8 0.8)
-				)
-				(justify left)
-			)
-		)
-		(property "Value" "0805,0"
-			(at 110.49 124.4599 0)
-			(effects
-				(font
-					(size 0.8 0.8)
-				)
-				(justify left)
-			)
-		)
-		(property "Footprint" "R_0805_2012Metric"
-			(at 107.95 123.19 0)
-			(effects
-				(font
-					(size 1.27 1.27)
-				)
-				(hide yes)
-			)
-		)
-		(property "Datasheet" "https://datasheet.lcsc.com/lcsc/2110251730_UNI-ROYAL-Uniroyal-Elec-0805W8F0000T5E_C17477.pdf"
-			(at 107.95 123.19 0)
-			(effects
-				(font
-					(size 1.27 1.27)
-				)
-				(hide yes)
-			)
-		)
-		(property "Description" "1% 125mW Thick Film Resistors 150V   800ppm    -55    155   0   0805 Chip Resistor - Surface Mount ROHS"
-			(at 107.95 123.19 0)
-			(effects
-				(font
-					(size 1.27 1.27)
-				)
-				(hide yes)
-			)
-		)
-		(property "LCSC" "C17477"
-			(at 107.95 123.19 0)
-			(effects
-				(font
-					(size 0.0254 0.0254)
-				)
-				(hide yes)
-			)
-		)
-		(property "MFG" "UNI-ROYAL(Uniroyal Elec)"
-			(at 107.95 123.19 0)
-			(effects
-				(font
-					(size 0.0254 0.0254)
-				)
-				(hide yes)
-			)
-		)
-		(property "MFGPN" "0805W8F0000T5E"
-			(at 107.95 123.19 0)
-			(effects
-				(font
-					(size 0.0254 0.0254)
-				)
-				(hide yes)
-			)
-		)
-		(pin "2"
-		)
-		(pin "1"
-		)
-		(instances
-			(project "MCUModule"
-				(path "/352d7abe-fc72-4473-8b68-62eecf44f496/c82070cb-20dc-4a3e-92d2-ca1724b01eaa"
-					(reference "R19")
-					(unit 1)
-				)
-				(path "/352d7abe-fc72-4473-8b68-62eecf44f496/7d8e5f80-7b11-4de4-ab98-83d2b8c6b4e1"
-					(reference "R10")
-					(unit 1)
-				)
-			)
-		)
-	)
-	(symbol
 		(lib_id "jlcpcb-basic-resistor:0805,10k")
 		(at 189.23 86.36 90)
@@
 			)
 		)
-		(property "Footprint" ""
+		(property "Footprint" "Package_DIP:DIP-16_W7.62mm_Socket"
 			(at 127 111.76 0)
 			(effects

Commit message: updated BOM
Parts:
- C2: value 0805,100nF,50V,X7R -> 100nF 50V,X7R; footprint C_0805_2012Metric -> Capacitor_SMD:C_0805_2012Metric; Digikey PN (none) -> 1276-1003-1-ND
- R11, R20, R3, R4, R5, R6, R7, R8, R9: value 0805,20k -> 20k; footprint R_0805_2012Metric -> Resistor_SMD:R_0805_2012Metric; Digikey PN (none) -> RMCF0805FT20K0CT-ND
- R12, R13, R14, R15, R16, R17, R18: value 0805,10k -> 10k; footprint R_0805_2012Metric -> Resistor_SMD:R_0805_2012Metric; Digikey PN (none) -> RMCF0805FT10K0CT-ND
- U6: Digikey PN (none) -> 296-33112-5-ND
