File: Rev A/MCUModule.kicad_sch (KiCad schematic)
At the start: 8 parts, among them U1 RaspberryPi_Pico, U2 74HC4051, U5 LM324

Commit message: added more schematic stuffs
Parts:
- added C5, C6: 0805,1uF,50V,X7R, C_0805_2012Metric, symbol jlcpcb-basic-capacitor:0805,1uF,50V,X7R
- added C7: 0805,100nF,50V,X7R, C_0805_2012Metric, symbol jlcpcb-basic-capacitor:0805,100nF,50V,X7R
- added R38: 0805,4.7k, R_0805_2012Metric, symbol jlcpcb-basic-resistor:0805,4.7k
- added R39, R40, R41, R42: 0805,10k, R_0805_2012Metric, symbol jlcpcb-basic-resistor:0805,10k
- added R43: 0805,27k, R_0805_2012Metric, symbol jlcpcb-basic-resistor:0805,27k
- added U4: LM7805_TO220, Package_TO_SOT_THT:TO-220-3_Vertical, symbol Regulator_Linear:LM7805_TO220
Connections:
- net GND: now also U5.11 (V-), C5.2, C6.2, C7.2, R39.2, R41.2, R42.2, U4.2 (GND)
- net at U5.12 (+): now also R42.1, R43.2
- net at U5.13 (-): now also R40.1, R41.1
- net at U5.14: now also R38.1
- net +5V: now reaches U5.4 (V+)
- net +5V: now also U1.39 (VSYS), C5.1, C7.1, R40.2, U4.3 (VO)
- net 12V_Wall_Bad: now reaches U1.24 (GPIO18)
- net 12V_Wall_Bad: now also R38.2, R39.1
- new net: C6.1, U4.1 (VI)
Other:
- moved on the sheet: R1, U1, U2, U5D, U5E

Commit message: Update MCUModule.kicad_sch
Parts:
- added C8, C9: 0805,100nF,50V,X7R, C_0805_2012Metric, symbol jlcpcb-basic-capacitor:0805,100nF,50V,X7R
- added D1, D2: 1N5819WS, Diode_SMD:D_SOD-323, symbol Diode:1N5819WS
- added J1: RJ45_Shielded, Connector_RJ:RJ45_Shielded_EthernetJack, symbol Connector:RJ45_Shielded
- added U7: 74HC14, symbol 74xx:74HC14
Connections:
- net +3.3V: now also U1.36 (3V3), C9.1
- net +5V: now also C8.1, U7.14 (VCC)
- net DATA_DISPLAY: now also U7.3
- net GND: now also C8.2, C9.2, J1.1, J1.SH, U7.7 (GND)
- net SRCLK_DISPLAY: now also U7.5
- net at C6.1, U4.1 (VI): now also D1.1 (K), D2.1 (K)
- net 12V_Wall: now reaches R43.1
- net 12V_Wall: now also D1.2 (A)
- net BoostVoltage_0.1x: now reaches U2.12 (A3)
- net LightISense1: now reaches U2.13 (A0)
- net LightISense2: now reaches U2.14 (A1)
- net brightnessKnob: now reaches U2.15 (A2)
- net at U1.34 (GPIO28_ADC2): no longer U2.3 (A)
- net DisableBackupPico: now reaches U1.12 (GPIO9)
- net PowerModuleEna1: now reaches U1.19 (GPIO14)
- net PowerModuleEna2: now reaches U1.20 (GPIO15)
- net AnalogMuxOut: now reaches U1.31 (GPIO26_ADC0)
- net AnalogMuxOut: now also U2.3 (A)
- net BoostEna1: now reaches U1.4 (GPIO2)
- net BoostEna2: now reaches U1.5 (GPIO3)
- net BatChgEna1: now reaches U1.6 (GPIO4)
- net BatChgEna2: now reaches U1.7 (GPIO5)
- net RCLK_DISPLAY renamed ~{RCLK_DISPLAY}
- net ~{RCLK_DISPLAY}: now also U7.9
- net ~{OE_DISPLAY} renamed OE_DISPLAY
- net OE_DISPLAY: now also U7.11
- new net: U7.1, U7.4
- new net: J1.7, U7.2
- new net: J1.4, U7.10
- new net: J1.6, U7.12
- new net: U7.13, U7.6
- new net: J1.5, U7.8
- new net +12V: J1.8
- new net 12V_Battery: D2.2 (A)
- new net DIM: J1.3
- no-connect marks 3 -> 4
Other:
- note added: "12V from Wall Brownout Interrupt Detection"
- note added: "5V LDO"
- note added: "Analog Mux"
- note added: "Line Driver and Ethernet port for User Display"
- note added: "Op Amp PWR"
- note added: "Pi Pico"
- note added: "RCLK and OE are inverted in this topology"
- note added: "Shift Register based DAC + Buffer for Buck Control"
- moved on the sheet: C3, C4, C5, C6, C7, R1, R36, R37, R38, R39, R40, R41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

Commit message: routed
Parts:
- removed R1: 0603,0, R_0603_1608Metric, symbol jlcpcb-basic-resistor:0603,0
- added D10, D11, D12, D13, D3, D4, D5, D6, D7, D8, D9: PESD3V3L1BA,115, Diode_SMD:D_SOD-323F, symbol Diode:SMAJ5.0CA
- added D14, D15, D17, D18: 1N5819WS, Diode_SMD:D_SOD-323, symbol Diode:1N5819WS
- added D16: SMAZ15Z-13-F, Diode_SMD:D_SMA, symbol Device:D_Zener_Small_Filled
- added H1, H2, H3, H4: M3 Hole, MountingHole:MountingHole_3.2mm_M3_Pad_TopBottom, symbol Mechanical:MountingHole_Pad
- added J2: 2x7 P2.54mm, Connector_PinHeader_2.54mm:PinHeader_2x07_P2.54mm_Vertical, symbol Connector_Generic:Conn_02x07_Odd_Even
- added Q1: 2SD1047, Package_TO_SOT_THT:TO-3PB-3_Vertical, symbol Transistor_BJT:2SD1047
- added R1: 0805,0, R_0805_2012Metric, symbol jlcpcb-basic-resistor:0805,0
- added R10, R19: 0805,10k, R_0805_2012Metric, symbol jlcpcb-basic-resistor:0805,10k
- added R44: 0805,33k, R_0805_2012Metric, symbol jlcpcb-basic-resistor:0805,33k
- J1: footprint Connector_RJ:RJ45_Shielded_EthernetJack -> Connectors_SurgicalLighting:CONN_A-2014-2S-4-N-R_ASM
- U2: footprint (none) -> Package_DIP:DIP-16_W7.62mm_Socket
- U5, U7: footprint (none) -> Package_DIP:DIP-14_W7.62mm_Socket
Connections:
- net 12V_Battery: now also D14.2 (A), H3.1
- net 12V_Wall: now also D15.2 (A), H4.1, R44.2
- net 12V_Wall_Bad: now also U1.16 (GPIO12); no longer U1.24 (GPIO18)
- net BatChgEna1: now also U1.11 (GPIO8), D4.2 (A2), J2.7 (Pin_7); no longer U1.6 (GPIO4)
- net BatChgEna2: now also U1.14 (GPIO10), D3.2 (A2), J2.9 (Pin_9); no longer U1.7 (GPIO5)
- net BoostEna1: now also U1.6 (GPIO4), D5.2 (A2), J2.3 (Pin_3); no longer U1.4 (GPIO2)
- net BoostEna2: now also U1.9 (GPIO6), D6.2 (A2), J2.5 (Pin_5); no longer U1.5 (GPIO3)
- net BoostVoltage_0.1x: no longer U2.12 (A3)
- net DATA_DAC: now also U1.20 (GPIO15); no longer U1.11 (GPIO8)
- net DATA_DISPLAY: now also U1.24 (GPIO18), U7.1; no longer U1.14 (GPIO10), U7.3
- net DIM: now also U2.12 (A3)
- net DisableBackupPico: now also U1.4 (GPIO2), D13.2 (A2), J2.2 (Pin_2); no longer U1.12 (GPIO9)
- net GND: now also U5.10 (+), D10.1 (A1), D11.1 (A1), D12.1 (A1), D13.1 (A1), D16.2 (A), D3.1 (A1), D4.1 (A1), D5.1 (A1), D6.1 (A1), D7.1 (A1), D8.1 (A1), D9.1 (A1), H1.1, J2.13 (Pin_13), J2.14 (Pin_14), R1.2, R19.1
- net OE_DISPLAY: now also U1.22 (GPIO17), U7.5; no longer U1.17 (GPIO13), U7.11
- net PWM_Lights1: now also U1.10 (GPIO7), D10.2 (A2), J2.8 (Pin_8); no longer U1.21 (GPIO16)
- net PWM_Lights2: now also U1.12 (GPIO9), D9.2 (A2), J2.10 (Pin_10); no longer U1.22 (GPIO17)
- net PowerModuleEna1: now also U1.5 (GPIO3), D12.2 (A2), J2.4 (Pin_4); no longer U1.19 (GPIO14)
- net PowerModuleEna2: now also U1.7 (GPIO5), D11.2 (A2), J2.6 (Pin_6); no longer U1.20 (GPIO15)
- net RCLK_DAC: now also U1.19 (GPIO14); no longer U1.9 (GPIO6)
- net RelaySelectHighPreference: now also U1.15 (GPIO11), D8.2 (A2), J2.12 (Pin_12); no longer U1.25 (GPIO19)
- net S0: now also U1.29 (GPIO22); no longer U1.26 (GPIO20)
- net S2: now also U1.26 (GPIO20); no longer U1.29 (GPIO22)
- net SRCLK_DAC: now also U1.17 (GPIO13); no longer U1.10 (GPIO7)
- net SRCLK_DISPLAY: now also U1.25 (GPIO19), U7.13; no longer U1.15 (GPIO11), U7.5
- net ~{RCLK_DISPLAY}: now also U1.21 (GPIO16); no longer U1.16 (GPIO12)
- net at C6.1, D1.1 (K), D2.1 (K)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: now also D18.1 (K)
- net at U5.1, U5.2 (-): now also R37.1; no longer R36.1
- net at U5.6 (-), U5.7: now also R36.1; no longer R37.1
- net DATA_5V: now reaches U7.4
- net DATA_5V: now also J1.7; no longer U7.1
- net at U7.2: now also U7.3; no longer J1.7
- net OE_5V: now reaches J1.4
- net OE_5V: now also U7.6; no longer U7.10
- net at U2.6 (~{E}): now also R1.1
- net at U5.8: now also U5.9 (-)
- net at U7.12: now also U7.11; no longer J1.6
- net RCLK_5V: now reaches J1.5, U7.8
- net ModuleENA: now reaches U1.30 (RUN)
- net ModuleENA: now also D7.2 (A2), J2.1 (Pin_1)
- net at U1.32 (GPIO27_ADC1): now also R19.2, R44.1
- net +12V: no longer names the net of J1.8
- net +12V: now also D14.1 (K), D15.1 (K), D17.1 (K)
- net brightnessKnob: no longer names the net of U2.15 (A2)
- new net: D16.1 (K), Q1.1 (B), R10.2
- new net 15V_SOLAR: D17.2 (A), D18.2 (A), Q1.3 (E)
- new net SOLAR: H2.1, Q1.2 (C), R10.1
- new net SRCLK_5V: J1.6, U7.10
- no-connect marks 4 -> 5
Other:
- note added: "Mounting Holes for Power Connections"
- moved on the sheet: C3, C4, R36, R37, U5C, U7A, U7B, U7C, U7E, U7F

Commit message: updated BOM
Parts:
- C3, C4, C5, C6: value 0805,1uF,50V,X7R -> 1uF 50V,X7R; footprint C_0805_2012Metric -> Capacitor_SMD:C_0805_2012Metric; Digikey PN (none) -> 1276-1029-1-ND
- C7, C8, C9: value 0805,100nF,50V,X7R -> 100nF 50V,X7R; footprint C_0805_2012Metric -> Capacitor_SMD:C_0805_2012Metric; Digikey PN (none) -> 1276-1003-1-ND
- D1, D14, D15, D17, D18, D2: Digikey PN (none) -> B5819WS-TPMSCT-ND
- D10, D11, D12, D13, D3, D4, D5, D6, D7, D8, D9: Digikey PN (none) -> 1727-3825-1-ND
- D16: Digikey PN (none) -> SMAZ15-FDICT-ND
- J1: Digikey PN (none) -> AE10399-ND
- J2: Digikey PN (none) -> 2057-PH2-14-UA-ND
- Q1: Digikey PN (none) -> 497-11320-5-ND
- R1: value 0805,0 -> 0; footprint R_0805_2012Metric -> Resistor_SMD:R_0805_2012Metric; Digikey PN (none) -> RMCF0805ZT0R00CT-ND
- R10, R19, R39, R40, R41, R42: value 0805,10k -> 10k; footprint R_0805_2012Metric -> Resistor_SMD:R_0805_2012Metric; Digikey PN (none) -> RMCF0805FT10K0CT-ND
- R36, R37: value 0805,1k -> 1k; footprint R_0805_2012Metric -> Resistor_SMD:R_0805_2012Metric; Digikey PN (none) -> RMCF0805FT1K00CT-ND
- R38: value 0805,4.7k -> 4.7k; footprint R_0805_2012Metric -> Resistor_SMD:R_0805_2012Metric; Digikey PN (none) -> RMCF0805FT4K70CT-ND
- R43: value 0805,27k -> 27k; footprint R_0805_2012Metric -> Resistor_SMD:R_0805_2012Metric; Digikey PN (none) -> RMCF0805FT27K0CT-ND
- R44: value 0805,33k -> 33k; footprint R_0805_2012Metric -> Resistor_SMD:R_0805_2012Metric; Digikey PN (none) -> RMCF0805FT33K0CT-ND
- U1: Digikey PN (none) -> 2648-SC0915CT-ND
- U2: Digikey PN (none) -> 296-12810-5-ND
- U4: Digikey PN (none) -> 2129-NJM7805FA-ND
- U5: Digikey PN (none) -> 296-1391-5-ND
- U7: Digikey PN (none) -> TC74HC14APF-ND
